File: Electronics/PCB/AstroPlant_ExtensionBoard/astroplant-extension-board-mk0-7/Astroplant_AL.kicad_pcb (KiCad board)
At the start: 2 copper layers, 88 parts, among them J1 JST_XH_Relays, J10 JST_XH_UART, J11 JST_HX_2, J12 JST-XH_LED_GND, J13 B5B-XH-A_LF__SN_, J16 JST_HX_2, J17 JST_HX_2, J18 JST_HX_2, J19 JST_HX_2, J2 2x40 2.5mm Header, J20 Conn_01x02, J21 Conn_01x02, J22 JST_XH_I2C, J23 JST_XH_I2C, J24 JST_XH_I2C, J25 JST_XH_I2C, J26 JST_XH_I2C, J27 JST_XH_I2C, J3 JST-XH_3, J4 JST-XH_3, J5 JST_HX_2, J6 629105136821, J7 JST-XH_3, J8 JST_HX_2, J9 JST-XH_3, Q1 IRLML6344TRPBF, Q2 IRLML6344TRPBF, Q3 IRLML6344TRPBF, Q4 IRLML6344TRPBF, Q5 IRLML6344TRPBF, SW1 SW_Push, SW2 SW_Push, SW3 SW_Push, SW4 SW_Push, U1 USBLC6-2SC6, U2 STM32WB55RGVx

Commit message: Place components on PCB
Parts:
- removed the D1 at (113.1, 82.2)
- removed J12: JST-XH_LED_GND, SamacSys_Parts:B4BXHALFSN
- removed the R13 at (120.7, 122.8)
- removed the R13 at (141.8, 65.2)
- removed the R6 at (89.0, 114.9)
- removed the R6 at (113.0, 84.8)
- added C13: 100pF, Capacitor_SMD:C_0603_1608Metric, F.Cu at (77.7, 118.4)
- added C14: 100nF, Capacitor_SMD:C_0603_1608Metric, F.Cu at (79.2, 118.4)
- added R13: 1k, Resistor_SMD:R_0603_1608Metric, F.Cu at (72.3, 119.2)
- added R6: 1k, Resistor_SMD:R_0603_1608Metric, F.Cu at (83.9, 100.1)
- C1, C10, C11, C12, C2, C5, C9: value 0.1uF -> 100nF; footprint Capacitor_SMD:C_0805_2012Metric -> Capacitor_SMD:C_0603_1608Metric
- R1, R12, R2, R24, R3, R4, R5, R7: value 10K -> 10k; footprint Resistor_SMD:R_0805_2012Metric -> Resistor_SMD:R_0603_1608Metric
- R10, R8, R9: value 100K -> 10k; footprint Resistor_SMD:R_0805_2012Metric -> Resistor_SMD:R_0603_1608Metric
- R11: footprint Resistor_SMD:R_0805_2012Metric -> Resistor_SMD:R_0603_1608Metric
- R14, R15, R16, R17, R18, R19, R20, R21, R22, R23: value 10K -> 1k; footprint Resistor_SMD:R_0805_2012Metric -> Resistor_SMD:R_0603_1608Metric
- moved SW1 70.2 mm to (121.8, 129.0), turned to 90 degrees
- moved SW4 68.2 mm to (118.0, 107.8), turned to 180 degrees
- moved R21 68.0 mm to (72.6, 85.6)
- moved SW2 66.7 mm to (130.1, 129.1), turned to 90 degrees
- moved SW3 65.3 mm to (138.7, 129.1), turned to 90 degrees
- moved C12 64.1 mm to (109.0, 107.3), turned to 90 degrees
- moved D1 63.9 mm to (109.1, 104.0), turned to -90 degrees
- moved J19 63.7 mm to (124.6, 69.7), turned to 180 degrees
- moved J18 63.2 mm to (116.0, 69.7), turned to 180 degrees
- moved J5 61.1 mm to (122.7, 117.1)
- moved C13 60.3 mm to (107.1, 94.9), turned to 90 degrees
- moved L1 60.0 mm to (57.4, 151.5)
- moved L2 60.0 mm to (57.4, 153.6)
- moved C6 60.0 mm to (70.9, 139.3)
- moved C7 60.0 mm to (70.9, 141.3)
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Connections:
- C1 pad 1: GND -> +3V3
- C1 pad 2: 5V_RPi -> GND
- C10 pad 1: GND -> +3V3
- C10 pad 2: +3V3 -> GND
- C11 pad 1: GND -> +3V3
- C11 pad 2: +3V3 -> GND
- C2 pad 1: GND -> 5V_RPi
- C2 pad 2: +3V3 -> GND
- C5 pad 1: GND -> +3V3
- C5 pad 2: +3V3 -> GND
- C9 pad 1: GND -> +3V3
- C9 pad 2: +3V3 -> GND
- R1 pad 1: +3V3 -> SCL_5V
- R1 pad 2: SDA -> +5V
- R10 pad 1: GPIO16 -> GND
- R10 pad 2: GND -> GPIO16
- R11 pad 1: +5V -> Net-(D5-A)
- R11 pad 2: Net-(D5-A) -> +5V
- R12 pad 1: Net-(J6-Pad4) -> GND
- R12 pad 2: GND -> Net-(J6-Pad4)
- R15 pad 1: Net-(U2-PA2) -> Net-(U2-PA0)
- R15 pad 2: GPIO20 -> GPIO13
- R16 pad 1: GPIO24 -> GPIO27
- R16 pad 2: Net-(U2-PC12) -> Net-(U2-PC15)
- R17 pad 1: GPIO25 -> GPIO26
- R17 pad 2: Net-(U2-PC13) -> Net-(U2-PC14)
- R18 pad 1: GPIO26 -> GPIO25
- R18 pad 2: Net-(U2-PC14) -> Net-(U2-PC13)
- R19 pad 1: GPIO27 -> GPIO24
- R19 pad 2: Net-(U2-PC15) -> Net-(U2-PC12)
- R2 pad 1: +5V -> SCL
- R2 pad 2: SDA_5V -> +3V3
- R20 pad 1: GPIO23 -> GPIO4
- R20 pad 2: Net-(U2-PC11) -> Net-(U2-PC5)
- R21 pad 1: GPIO22 -> GPIO17
- R21 pad 2: Net-(U2-PC10) -> Net-(U2-PC6)
- R22 pad 1: GPIO17 -> GPIO22
- R22 pad 2: Net-(U2-PC6) -> Net-(U2-PC10)
- R23 pad 1: GPIO4 -> GPIO23
- R23 pad 2: Net-(U2-PC5) -> Net-(U2-PC11)
- R3 pad 1: +3V3 -> SDA
- R3 pad 2: SCL -> +3V3
- R4 pad 1: +5V -> SDA_5V
- R4 pad 2: SCL_5V -> +5V
- R5 pad 1: +3V3 -> GPIO17
- R5 pad 2: GPIO17 -> +3V3
- R7 pad 1: +3V3 -> GPIO4
- R7 pad 2: GPIO4 -> +3V3
- R8 pad 1: GPIO12 -> GND
- R8 pad 2: GND -> GPIO12
- R9 pad 1: GPIO19 -> GND
- R9 pad 2: GND -> GPIO19
- U2 pad 1: +3V3 -> unconnected-(U2-VBAT-Pad1)
Routing:
- net (no net): vias 0 -> 6
Other:
- board outline added: 100 x 65 mm
