File: Electronics/PCB/AstroPlant_ExtensionBoard/astroplant-extension-board-mk0-7/I2C_Interface.kicad_sch (KiCad schematic)
At the start: 6 parts, among them J22 JST_XH_I2C, J23 JST_XH_I2C, J24 JST_XH_I2C, J25 JST_XH_I2C, J26 JST_XH_I2C, J27 JST_XH_I2C

Commit message: Update schematic and change library path
Parts:
- J22, J23, J24, J25, J26, J27: footprint Connector_JST:JST_XH_B04B-XH-A_1x04_P2.50mm_Vertical -> SamacSys_Parts:B4BXHALFSN
Changed lines of the file:
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@@
       (effects (font (size 1.524 1.524)))
     )
-    (property "Footprint" "Connector_JST:JST_XH_B04B-XH-A_1x04_P2.50mm_Vertical" (at 95.25 92.71 0)
+    (property "Footprint" "SamacSys_Parts:B4BXHALFSN" (at 95.25 92.71 0)
       (effects (font (size 1.524 1.524)) hide)
     )
@@
       (effects (font (size 1.524 1.524)))
     )
-    (property "Footprint" "Connector_JST:JST_XH_B04B-XH-A_1x04_P2.50mm_Vertical" (at 93.98 124.46 0)
+    (property "Footprint" "SamacSys_Parts:B4BXHALFSN" (at 93.98 124.46 0)
       (effects (font (size 1.524 1.524)) hide)
     )
@@
       (effects (font (size 1.524 1.524)))
     )
-    (property "Footprint" "Connector_JST:JST_XH_B04B-XH-A_1x04_P2.50mm_Vertical" (at 158.75 123.19 0)
+    (property "Footprint" "SamacSys_Parts:B4BXHALFSN" (at 158.75 123.19 0)
       (effects (font (size 1.524 1.524)) hide)
     )
@@
       (effects (font (size 1.524 1.524)))
     )
-    (property "Footprint" "Connector_JST:JST_XH_B04B-XH-A_1x04_P2.50mm_Vertical" (at 223.52 123.19 0)
+    (property "Footprint" "SamacSys_Parts:B4BXHALFSN" (at 223.52 123.19 0)
       (effects (font (size 1.524 1.524)) hide)
     )
@@
       (effects (font (size 1.524 1.524)))
     )
-    (property "Footprint" "Connector_JST:JST_XH_B04B-XH-A_1x04_P2.50mm_Vertical" (at 224.79 91.44 0)
+    (property "Footprint" "SamacSys_Parts:B4BXHALFSN" (at 224.79 91.44 0)
       (effects (font (size 1.524 1.524)) hide)
     )
@@
       (effects (font (size 1.524 1.524)))
     )
-    (property "Footprint" "Connector_JST:JST_XH_B04B-XH-A_1x04_P2.50mm_Vertical" (at 160.02 91.44 0)
-      (effects (font (size 1.524 1.524)) hide)
-    )
+    (property "Footprint" "SamacSys_Parts:B4BXHALFSN" (at 160.02 91.44 0)
+      (effects (font (size 1.524 1.524)) hide)
+    )

Commit message: Updated PCB from a backup save to solve issue with git
Parts:
- J22, J23, J24, J25, J26, J27: value JST_XH_I2C -> B4B-XH-A(LF)(SN)
Changed lines of the file:
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@@
       (effects (font (size 1.524 1.524)))
     )
-    (property "Value" "JST_XH_I2C" (at 100.33 78.74 90)
+    (property "Value" "B4B-XH-A(LF)(SN) " (at 100.33 78.74 90)
       (effects (font (size 1.524 1.524)))
     )
@@
       (effects (font (size 1.524 1.524)))
     )
-    (property "Value" "JST_XH_I2C" (at 99.06 110.49 90)
+    (property "Value" "B4B-XH-A(LF)(SN) " (at 99.06 110.49 90)
       (effects (font (size 1.524 1.524)))
     )
@@
       (effects (font (size 1.524 1.524)))
     )
-    (property "Value" "JST_XH_I2C" (at 163.83 109.22 90)
+    (property "Value" "B4B-XH-A(LF)(SN) " (at 163.83 109.22 90)
       (effects (font (size 1.524 1.524)))
     )
@@
       (effects (font (size 1.524 1.524)))
     )
-    (property "Value" "JST_XH_I2C" (at 228.6 109.22 90)
+    (property "Value" "B4B-XH-A(LF)(SN) " (at 228.6 109.22 90)
       (effects (font (size 1.524 1.524)))
     )
@@
       (effects (font (size 1.524 1.524)))
     )
-    (property "Value" "JST_XH_I2C" (at 229.87 77.47 90)
+    (property "Value" "B4B-XH-A(LF)(SN) " (at 229.87 77.47 90)
       (effects (font (size 1.524 1.524)))
     )
@@
       (effects (font (size 1.524 1.524)))
     )
-    (property "Value" "JST_XH_I2C" (at 165.1 77.47 90)
-      (effects (font (size 1.524 1.524)))
-    )
+    (property "Value" "B4B-XH-A(LF)(SN) " (at 165.1 77.47 90)
+      (effects (font (size 1.524 1.524)))
+    )
