File: Electronics/PCB/AstroPlant_ExtensionBoard/astroplant-extension-board-mk0-7/outputs.kicad_sch (KiCad schematic)
At the start: 14 parts, among them J13 B5B-XH-A_LF__SN_, J16 JST_HX_2, J17 JST_HX_2, J18 JST_HX_2, J19 JST_HX_2, Q3 IRLML6344TRPBF, Q4 IRLML6344TRPBF, Q5 IRLML6344TRPBF

Commit message: Updated PCB from a backup save, solve issues of the 1st prototype
Parts:
- D2, D3, D4: value S1A -> S1A-13-F
- J13: value B5B-XH-A_LF__SN_ -> B5B-XH-A(LF)(SN)
- J16, J17, J18, J19: value JST_HX_2 -> B2B-XH-A(LF)(SN)
- R24, R25: value 10k -> GPR060310K; MPN CRCW060310K0DHEAP -> GPR060310K
Changed lines of the file:
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@@
       (effects (font (size 1.27 1.27)))
     )
-    (property "Value" "S1A" (at 67.31 113.03 0)
+    (property "Value" "S1A-13-F" (at 67.31 113.03 0)
       (effects (font (size 1.27 1.27)))
     )
@@
       (effects (font (size 1.27 1.27)))
     )
-    (property "Value" "S1A" (at 130.81 113.03 0)
+    (property "Value" "S1A-13-F" (at 130.81 113.03 0)
       (effects (font (size 1.27 1.27)))
     )
@@
       (effects (font (size 1.27 1.27)))
     )
-    (property "Value" "S1A" (at 194.31 115.57 0)
+    (property "Value" "S1A-13-F" (at 194.31 115.57 0)
       (effects (font (size 1.27 1.27)))
     )
@@
       (effects (font (size 1.524 1.524)))
     )
-    (property "Value" "JST_HX_2" (at 213.36 119.38 0)
+    (property "Value" "B2B-XH-A(LF)(SN) " (at 213.36 119.38 0)
       (effects (font (size 1.524 1.524)))
     )
@@
       (effects (font (size 1.524 1.524)))
     )
-    (property "Value" "JST_HX_2" (at 229.87 119.38 0)
+    (property "Value" "B2B-XH-A(LF)(SN) " (at 229.87 119.38 0)
       (effects (font (size 1.524 1.524)))
     )
@@
       (effects (font (size 1.524 1.524)))
     )
-    (property "Value" "JST_HX_2" (at 149.86 118.11 0)
+    (property "Value" "B2B-XH-A(LF)(SN) " (at 149.86 118.11 0)
       (effects (font (size 1.524 1.524)))
     )
@@
       (effects (font (size 1.524 1.524)))
     )
-    (property "Value" "JST_HX_2" (at 86.36 118.11 0)
+    (property "Value" "B2B-XH-A(LF)(SN) " (at 86.36 118.11 0)
       (effects (font (size 1.524 1.524)))
     )
@@
       (effects (font (size 1.27 1.27)) (justify left))
     )
-    (property "Value" "B5B-XH-A_LF__SN_" (at 168.91 71.12 0)
+    (property "Value" "B5B-XH-A(LF)(SN)" (at 168.91 71.12 0)
       (effects (font (size 1.27 1.27)) (justify left))
     )
@@
       (effects (font (size 1.27 1.27)) (justify right))
     )
-    (property "Value" "10k" (at 187.96 137.16 0)
+    (property "Value" "GPR060310K" (at 187.96 137.16 0)
       (effects (font (size 1.27 1.27)) (justify right))
     )
@@
       (effects (font (size 1.27 1.27)) hide)
     )
-    (property "MPN" "CRCW060310K0DHEAP" (at 185.42 135.89 0)
+    (property "MPN" "GPR060310K" (at 185.42 135.89 0)
       (effects (font (size 1.27 1.27)) hide)
     )
@@
       (effects (font (size 1.27 1.27)) (justify right))
     )
-    (property "Value" "10k" (at 124.46 134.62 0)
+    (property "Value" "GPR060310K" (at 124.46 134.62 0)
       (effects (font (size 1.27 1.27)) (justify right))
     )
@@
       (effects (font (size 1.27 1.27)) hide)
     )
-    (property "MPN" "CRCW060310K0DHEAP" (at 121.92 133.35 0)
+    (property "MPN" "GPR060310K" (at 121.92 133.35 0)
       (effects (font (size 1.27 1.27)) hide)
     )
@@
       (effects (font (size 1.27 1.27)) (justify right))
     )
-    (property "Value" "10k" (at 60.96 134.62 0)
+    (property "Value" "GPR060310K" (at 60.96 134.62 0)
       (effects (font (size 1.27 1.27)) (justify right))
     )
@@
       (effects (font (size 1.27 1.27)) hide)
     )
-    (property "MPN" "CRCW060310K0DHEAP" (at 58.42 133.35 0)
-      (effects (font (size 1.27 1.27)) hide)
-    )
+    (property "MPN" "GPR060310K" (at 58.42 133.35 0)
+      (effects (font (size 1.27 1.27)) hide)
+    )
