File: Electronics/PCB/AstroPlant_ExtensionBoard/astroplant-extension-board-mk0-7/Microcontroller.kicad_sch (KiCad schematic)
At the start: 44 parts, among them J12 CONUFL001-SMD-T, J15 ZX62D-B-5PA8(30), SW2 430156043726, SW3 430156043726, U1 USBLC6-2SC6, U2 STM32WB55RGV6, Y1 NX2016SA-32M-EXS00A-CS06465

Commit message: Fix the antenna (Implies a change in PCB routing)+ improve readme (add a tutorial to make the board on eurocicruit).
Parts:
- removed AE1: Antenna, RF_Antenna:Texas_SWRA117D_2.4GHz_Left, symbol Device:Antenna
- removed C19, C20, C21, C6: GRM1555C1H1R2WA01D, SamacSys_Parts:CAPC1005X55N, symbol SamacSys_Parts:GRM1555C1H1R2WA01D
- removed C7: GRM1555C1HR30WA01D, SamacSys_Parts:CAPC1005X55N, symbol SamacSys_Parts:GRM1555C1HR30WA01D
- removed C8: GRM1555C1HR80BA01D, SamacSys_Parts:CAPC1005X55N, symbol SamacSys_Parts:GRM1555C1HR80BA01D
- removed FL1: DEA162450BT-1260B2, DEA162450BT1295A1, symbol SamacSys_Parts:DEA162450BT-1260B2
- removed J12: CONUFL001-SMD-T, CONUFL001-SMD, symbol SamacSys_Parts:CONUFL001-SMD-T
- removed L1, L3: LQG15HS3N6S02D, SamacSys_Parts:LQG15WH0N7B02D, symbol SamacSys_Parts:LQG15HS3N6S02D
- removed L2: LQG15HS2N7S02J, SamacSys_Parts:LQG15WH0N7B02D, symbol SamacSys_Parts:LQG15HS2N7S02J
- removed R25, R26: GPR06030R, Resistor_SMD:R_0603_1608Metric, symbol Device:R_Small
- added C6, C7: GPC0603475-10, Capacitor_SMD:C_0603_1608Metric, symbol Device:C_Small
- added C8: GPC0603101, Capacitor_SMD:C_0603_1608Metric, symbol Device:C_Small
- added FL2: MLPF-WB55-01E3, MLPFWB5501E3, symbol SamacSys_Parts:MLPF-WB55-01E3
- added J6: 60312202114509, SamacSys_Parts:60312202114509, symbol SamacSys_Parts:60312202114509
- added L1: LBR2012T100K, Inductor_SMD:L_0805_2012Metric, symbol Device:L
- D1: value BAT54KFILM -> RB521S30T1G; Arrow Price/Stock https://www.arrow.com/en/products/bat54kfilm/stmicroelectro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 -> (none); MPN BAT54KFILM -> RB521S30T1G; Manufacturer_Name STMicroelectronics -> (none); Manufacturer_Part_Number BAT54KFILM -> (none); Mouser Part Number 511-BAT54KFILM -> (none); Mouser Price/Stock https://www.mouser.co.uk/ProductDetail/STMicroelectronics/B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 -> (none)
- R27: value CRCW0603180RFKEA -> GPR0603180R; MPN CRCW0603180RFKEA -> GPR0603180R
- Y1: MPN (none) -> NX2016SA-32M-EXS00A-CS06465
Connections:
- net +3V3: now also U2.1 (VBAT), C7.2, C8.1; no longer U2.41 (VFBSMPS), U2.43 (VLXSMPS)
- net GND: now also C6.1, C7.1, C8.2, FL2.2 (GND4), FL2.4 (GND1), FL2.5 (GND2), FL2.6 (GND3), J6.1 (In), J6.3 (GND), J6.4 (GND), J6.5 (GND)
- net Ant_62Ohm: now reaches U2.31 (RF1)
- net Ant_62Ohm: now also FL2.3 (IN)
- new net: C6.2, L1.1, U2.41 (VFBSMPS)
- new net: L1.2, U2.43 (VLXSMPS)
- new net Ant_50Ohm: FL2.1 (OUT), J6.2 (GND)
Other:
- moved on the sheet: Y1
